Commit message: modified world joint behavior in pr2.urdf.xacro to speed up testing cycle

File: pr2_robot/urdf/pr2.urdf.xacro (robot description, xacro)
@@ -602,5 +602,5 @@
     <origin xyz="0 0 0" rpy="0 0 0" />
     <axis xyz="0 0 1"/>
-    <limit effort="10000" velocity="0.1"/>
+    <limit effort="14000" velocity="0.2"/>
     <child link="base_footprint" />
     <parent link="world"/>
